File: PWMGenerator-aja/_autosave-PWMGenerator-aja.kicad_sch (KiCad schematic)
At the start: 30 parts, among them J1 Conn_01x03_Pin, Q1 NPN, Q2 NPN, Q3 PNP, Q4 PNP, SW1 SW_SPST, U1 LM7805_TO220, U2 LM339

Commit message: Finished Schematic A
Symbols and connections.
Parts:
- Q4: footprint (none) -> Package_TO_SOT_THT:TO-92_Inline; symbol Simulation_SPICE:PNP -> Transistor_BJT:2N3906
Connections:
- net VCC: now also Q4.1 (E); no longer Q4.3 (E)
- net at J1.2 (Pin_2), R10.1: now also Q4.3 (C); no longer Q4.1 (C)
Other:
- moved on the sheet: C1, C2, C3, D1, D2, D3, D4, D5, D6, F1, J1, Q1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
