File: PWMGenerator-aja/A Solution/PWMGenerator-aja.kicad_sch (KiCad schematic)
At the start: 30 parts, among them J1 Conn_01x03_Pin, Q1 NPN, Q2 NPN, Q3 PNP, Q4 PNP, SW1 SW_SPST, U1 LM7805_TO220, U2 LM339

Commit message: Rev 0.4.  Release version of A solution. Updated PCB Project A notes.
Parts:
- Q4: symbol Transistor_BJT:2N3906 -> Simulation_SPICE:PNP
Connections:
- net VCC: now also Q4.3 (E); no longer Q4.1 (E)
- net at J1.2 (Pin_2), R10.1: now also Q4.1 (C); no longer Q4.3 (C)
Changed lines of the file:
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@@
 		(title "CMPE2150 PWM Generator - aja")
 		(date "2024-12-03")
-		(rev "0.2")
+		(rev "0.4")
 		(company "NAIT CNT")
 		(comment 1 "Author: AJ Armstrong")
@@
 	)
 	(junction
+		(at 115.57 63.5)
+		(diameter 0)
+		(color 0 0 0 0)
+	)
+	(junction
 		(at 40.64 114.3)
 		(diameter 0)
@@
 	(wire
 		(pts
+			(xy 115.57 63.5) (xy 121.92 63.5)
+		)
+		(stroke
+			(width 0)
+			(type default)
+		)
+	)
+	(wire
+		(pts
 			(xy 144.78 92.71) (xy 170.18 92.71)
 		)
@@
 	(wire
 		(pts
+			(xy 115.57 59.69) (xy 115.57 63.5)
+		)
+		(stroke
+			(width 0)
+			(type default)
+		)
+	)
+	(wire
+		(pts
 			(xy 77.47 63.5) (xy 81.28 63.5)
 		)
@@
 	(wire
 		(pts
-			(xy 106.68 63.5) (xy 121.92 63.5)
+			(xy 106.68 63.5) (xy 115.57 63.5)
 		)
 		(stroke
@@
 			(width 0)
 			(type default)
+		)
+	)
+	(symbol
+		(lib_id "power:PWR_FLAG")
+		(at 115.57 59.69 0)
+		(unit 1)
+		(exclude_from_sim no)
+		(in_bom yes)
+		(on_board yes)
+		(dnp no)
+		(fields_autoplaced yes)
+		(property "Reference" "#FLG05"
+			(at 115.57 57.785 0)
+			(effects
+				(font
+					(size 1.27 1.27)
+				)
+				(hide yes)
+			)
+		)
+		(property "Value" "PWR_FLAG"
+			(at 115.57 54.61 0)
+			(effects
+				(font
+					(size 1.27 1.27)
+				)
+			)
+		)
+		(property "Footprint" ""
+			(at 115.57 59.69 0)
+			(effects
+				(font
+					(size 1.27 1.27)
+				)
+				(hide yes)
+			)
+		)
+		(property "Datasheet" "~"
+			(at 115.57 59.69 0)
+			(effects
+				(font
+					(size 1.27 1.27)
+				)
+				(hide yes)
+			)
+		)
+		(property "Description" "Special symbol for telling ERC where power comes from"
+			(at 115.57 59.69 0)
+			(effects
+				(font
+					(size 1.27 1.27)
+				)
+				(hide yes)
+			)
+		)
+		(pin "1"
+		)
+		(instances
+			(project "PWMGenerator-aja"
+				(path "/18199a25-5472-4b5c-b90a-fcfdecd0a2ee"
+					(reference "#FLG05")
+					(unit 1)
+				)
+			)
 		)
 	)
@@
 	)
 	(symbol
-		(lib_id "Transistor_BJT:2N3906")
+		(lib_id "Simulation_SPICE:PNP")
 		(at 218.44 82.55 0)
 		(mirror x)
@@
 		)
 		(property "Footprint" "Package_TO_SOT_THT:TO-92_Inline"
-			(at 223.52 80.645 0)
-			(effects
-				(font
-					(size 1.27 1.27)
-					(italic yes)
-				)
-				(justify left)
-				(hide yes)
-			)
-		)
-		(property "Datasheet" "https://www.onsemi.com/pub/Collateral/2N3906-D.PDF"
+			(at 254 82.55 0)
+			(effects
+				(font
+					(size 1.27 1.27)
+				)
+				(hide yes)
+			)
+		)
+		(property "Datasheet" "https://ngspice.sourceforge.io/docs/ngspice-html-manual/manual.xhtml#cha_BJTs"
+			(at 254 82.55 0)
+			(effects
+				(font
+					(size 1.27 1.27)
+				)
+				(hide yes)
+			)
+		)
+		(property "Description" "Bipolar transistor symbol for simulation only, substrate tied to the emitter"
 			(at 218.44 82.55 0)
 			(effects
-				(font
-					(size 1.27 1.27)
-				)
-				(justify left)
-				(hide yes)
-			)
-		)
-		(property "Description" "-0.2A Ic, -40V Vce, Small Signal PNP Transistor, TO-92"
-			(at 218.44 82.55 0)
-			(effects
