File: PCB Makeup Project/PCB Makeup Project.kicad_sch (KiCad schematic)
At the start: 11 parts, among them J1 Conn_01x04_Pin, Q1 2N3906, SW1 Trigger, U2 TLC555xD, U3 LM324

Commit message: Bup
Parts:
- Q1: footprint Package_TO_SOT_THT:TO-92_Inline -> Package_TO_SOT_THT:TO-92
- U1: renamed from U3; footprint (none) -> Package_SO:TSSOP-14_4.4x5mm_P0.65mm
- renumbered SW1 to S1
Other:
- company: (none) -> NAIT CNT
- title: (none) -> CMPE2150 Pulse Generator - aja
Changed lines of the file:
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@@
 	(generator "eeschema")
 	(generator_version "9.0")
-	(paper "A4")
+	(paper "USLetter")
+	(title_block
+		(title "CMPE2150 Pulse Generator - aja")
+		(date "2025-05-17")
+		(rev "0")
+		(company "NAIT CNT")
+		(comment 1 "AJ Armstrong")
+	)
 	(junction
 		(at 139.7 135.89)
@@
 		(dnp no)
 		(fields_autoplaced yes)
-		(property "Reference" "U3"
+		(property "Reference" "U1"
 			(at 53.34 177.8 0)
 			(effects
@@
 			)
 		)
-		(property "Footprint" ""
+		(property "Footprint" "Package_SO:TSSOP-14_4.4x5mm_P0.65mm"
 			(at 52.07 190.5 0)
 			(effects
@@
 			(project ""
 				(path "/a64b8690-09f4-458e-8a6e-93d81a873170"
-					(reference "U3")
+					(reference "U1")
 					(unit 4)
 				)
@@
 			)
 		)
-		(property "Footprint" "Package_TO_SOT_THT:TO-92_Inline"
+		(property "Footprint" "Package_TO_SOT_THT:TO-92"
 			(at 142.24 80.645 0)
 			(effects
@@
 		(dnp no)
 		(fields_autoplaced yes)
-		(property "Reference" "U3"
+		(property "Reference" "U1"
 			(at 115.57 81.2799 0)
 			(effects
@@
 			)
 		)
-		(property "Footprint" ""
+		(property "Footprint" "Package_SO:TSSOP-14_4.4x5mm_P0.65mm"
 			(at 115.57 80.01 0)
 			(effects
@@
 			(project ""
 				(path "/a64b8690-09f4-458e-8a6e-93d81a873170"
-					(reference "U3")
+					(reference "U1")
 					(unit 5)
 				)
@@
 		(dnp no)
 		(fields_autoplaced yes)
-		(property "Reference" "SW1"
+		(property "Reference" "S1"
 			(at 55.88 123.19 0)
 			(effects
@@
 			(project ""
 				(path "/a64b8690-09f4-458e-8a6e-93d81a873170"
-					(reference "SW1")
+					(reference "S1")
 					(unit 1)
 				)
@@
 		(dnp no)
 		(fields_autoplaced yes)
-		(property "Reference" "U3"
+		(property "Reference" "U1"
 			(at 27.94 177.8 0)
 			(effects
@@
 			)
 		)
-		(property "Footprint" ""
+		(property "Footprint" "Package_SO:TSSOP-14_4.4x5mm_P0.65mm"
 			(at 26.67 190.5 0)
 			(effects
@@
 			(project ""
 				(path "/a64b8690-09f4-458e-8a6e-93d81a873170"
-					(reference "U3")
+					(reference "U1")
 					(unit 3)
 				)
@@
 		(on_board yes)
 		(dnp no)
-		(property "Reference" "U3"
+		(property "Reference" "U1"
 			(at 109.474 46.99 0)
 			(effects
@@
 			)
 		)
-		(property "Footprint" ""
+		(property "Footprint" "Package_SO:TSSOP-14_4.4x5mm_P0.65mm"
 			(at 106.68 57.15 0)
 			(effects
@@
 			(project ""
 				(path "/a64b8690-09f4-458e-8a6e-93d81a873170"
-					(reference "U3")
+					(reference "U1")
 					(unit 1)
 				)
@@
 		(on_board yes)
 		(dnp no)
-		(property "Reference" "U3"
+		(property "Reference" "U1"
 			(at 118.872 75.184 0)
 			(effects
@@
 			)
 		)
-		(property "Footprint" ""
+		(property "Footprint" "Package_SO:TSSOP-14_4.4x5mm_P0.65mm"
 			(at 115.57 85.09 0)
 			(effects
@@
 			(project ""
 				(path "/a64b8690-09f4-458e-8a6e-93d81a873170"
-					(reference "U3")
+					(reference "U1")
 					(unit 2)
 				)
